Commit message: robot model v2 after adversarial review: three solids and the knee motor re-booked by bolt pattern (thigh 2.76 / shin 3.36 kg), bearing split by joint axis, right-leg roll axes mirrored, CAD stops (knee -120, ankle +30), upper lump at the hip (CoM +63 mm like the old model - the 'more balanced' claim retracted), hip collision primitives within the contact budget
Co-Authored-By: Claude Opus 5 <noreply@anthropic.com>

File: pygmalion_locomotion/assets/pygmalion_v2/pygmalion_v2.urdf (robot description, URDF)
Before this commit: robot pygmalion_v2, 13 links, 12 joints
Links:
- link L_hip_pitch_link: mass 2.2854 -> 2.1779
- link L_hip_roll_link: mass 1.6064 -> 1.8198
- link L_shin_link: mass 4.7588 -> 3.3628
- link L_thigh_link: mass 1.5496 -> 2.7562
- link R_hip_pitch_link: mass 2.2854 -> 2.1779
- link R_hip_roll_link: mass 1.6064 -> 1.8198
- link R_shin_link: mass 4.7588 -> 3.3628
- link R_thigh_link: mass 1.5496 -> 2.7562
- link base_link: mass 19.314 -> 21.592
Joints:
- joint L_ankle_pitch_joint: limit lower=-0.872665 upper=0.698132 effort=90 velocity=20 -> lower=-0.872665 upper=0.523599 effort=90 velocity=20
- joint L_knee_joint: limit lower=-2.44346 upper=0.0 effort=120 velocity=20 -> lower=-2.094395 upper=0.0 effort=120 velocity=20
- joint R_ankle_pitch_joint: limit lower=-0.872665 upper=0.698132 effort=90 velocity=20 -> lower=-0.872665 upper=0.523599 effort=90 velocity=20
- joint R_ankle_roll_joint: axis -1 0 0 -> 1 0 0
- joint R_hip_roll_joint: axis 1 0 0 -> -1 0 0
- joint R_knee_joint: limit lower=-2.44346 upper=0.0 effort=120 velocity=20 -> lower=-2.094395 upper=0.0 effort=120 velocity=20

Commit message: robot model v2 round 2: the pelvis is mirrored where the STEP is one-sided (+0.17 kg, COM centred), ankle cross carries its bearings, validator fingerprints the L/R convention by foot rotation instead of point displacement, 61-point sweeps put the self-contact onsets at 11 deg adduction and -120 deg flexion
Co-Authored-By: Claude Opus 5 <noreply@anthropic.com>

File: pygmalion_locomotion/assets/pygmalion_v2/pygmalion_v2.urdf (robot description, URDF)
Before this commit: robot pygmalion_v2, 13 links, 12 joints
Links:
- link L_ankle_pitch_link: mass 0.066987 -> 0.086895
- link L_foot_link: mass 0.78529 -> 0.77534
- link L_shin_link: mass 3.3628 -> 3.3529
- link R_ankle_pitch_link: mass 0.066987 -> 0.086895
- link R_foot_link: mass 0.78529 -> 0.77534
- link R_shin_link: mass 3.3628 -> 3.3529
- link base_link: mass 21.592 -> 21.763

Commit message: v3: mass and inertia now come from Fusion 360 over MCP, not the STEP export - the live doc is a newer revision that carries the upper body, so the robot is 50.31 kg with a measured 22.09 kg torso instead of a 16.11 kg placeholder; every motor is confirmed a steel-density placeholder at the source; the bearing geometry confirms all six joint axes unchanged; and a pin named CenterPin_RS03 was substring-matched into a phantom 1.76 kg on the thigh before the Robstride guard
Co-Authored-By: Claude Opus 5 <noreply@anthropic.com>

File: pygmalion_locomotion/assets/pygmalion_v2/pygmalion_v2.urdf (robot description, URDF)
Before this commit: robot pygmalion_v2, 13 links, 12 joints
Links:
- link L_ankle_pitch_link: mass 0.086895 -> 0.087149
- link L_foot_link: mass 0.77534 -> 1.0326
- link L_hip_pitch_link: mass 2.1779 -> 2.1718
- link L_hip_roll_link: mass 1.8198 -> 1.6093
- link L_shin_link: mass 3.3529 -> 3.6275
- link L_thigh_link: mass 2.7562 -> 2.8959
- link R_ankle_pitch_link: mass 0.086895 -> 0.087149
- link R_foot_link: mass 0.77534 -> 1.0326
- link R_hip_pitch_link: mass 2.1779 -> 2.1718
- link R_hip_roll_link: mass 1.8198 -> 1.6093
- link R_shin_link: mass 3.3529 -> 3.6275
- link R_thigh_link: mass 2.7562 -> 2.8959
- link base_link: mass 21.763 -> 27.461

Commit message: CAD placeholders weigh what the real parts weigh, joint ranges measured, upper body modelled
Four things the user asked for, in one pass over the Fusion document.

MASS. Every motor and bearing in the CAD was still a stand-in solid at the default Steel
7850, so the model carried 13.695 kg of placeholders where the catalogue says 11.171. Their
density is now scaled per part until each weighs its manufacturer figure
(tools/fusion/set_placeholder_density.py, dry run by default). Three real errors fell out:
one 6810ZZ was modelled in ALUMINIUM (16.5 g for a 50 g bearing); RS02 is 380 g in the
manual, not the 405 g that circulates from resellers; and the JMC-JS06 placeholders are
spherical-bearing INSERTS at 12.83 g, within 1.3 % of THK's PB6, not the 35 g rod ends the
research had assumed - applying that estimate would have put 176 g of phantom mass on the
ankle ends. Measuring the placeholder before trusting the catalogue also overturned the
"RS04 is a shrunken solid" verdict: its bbox is 120.0 x 120.0 x 55.7 mm against a catalogue
120 x 120 x 56, so it is a hollow shell at the right envelope and density scaling is sound.

RANGE. rom_check.py turns each joint in the assembled CAD until two solids that were not
already touching push into each other. Getting a number worth trusting took three rewrites,
each recorded in docs/88: excluding whole body pairs hid the knee's own stop; convex hulls
filled in the yokes and reported 105 mm of built-in interference (real triangle meshes bring
that to 5.1 mm); and pairs the swept joint does not actually move had to be filtered out.

UPPER BODY. Torso, shoulder link and arm come out of Fusion with their meshes, on the three
axes the CAD has. Whole robot 42.098 kg, pelvis 5.166 + torso 5.966 + 11.464 per leg +
4.019 per arm side.

MCP. This Fusion build returns an empty message for anything a script prints, so payloads
now come back through the exception channel (no practical size cap, 200 KB verified). An
exception also ROLLS BACK the document edit, which silently reverted the density pass once -
mcp_client.run_script() exists for that.

docs/88_cad_placeholder_mass_rom.md, docs/raw/bearing-rodend-masses.md

Co-Authored-By: Claude Opus 4.8 <noreply@anthropic.com>

File: pygmalion_locomotion/assets/pygmalion_v2/pygmalion_v2.urdf (robot description, URDF)
Before this commit: robot pygmalion_v2, 13 links, 12 joints
Links:
- added link L_arm_link, mass 2.8414; collision mesh filename=meshes/arm_hull.stl; visual mesh filename=meshes/arm.stl
- added link L_shoulder_pitch_link, mass 1.1776; collision mesh filename=meshes/shoulder_pitch_link_hull.stl; visual mesh filename=meshes/shoulder_pitch_link.stl
- added link R_arm_link, mass 2.8414; collision mesh filename=meshes/R_arm_hull.stl; visual mesh filename=meshes/R_arm.stl
- added link R_shoulder_pitch_link, mass 1.1776; collision mesh filename=meshes/R_shoulder_pitch_link_hull.stl; visual mesh filename=meshes/R_shoulder_pitch_link.stl
- added link torso_link, mass 5.9658; collision mesh filename=meshes/torso_hull.stl; visual mesh filename=meshes/torso.stl
- link L_ankle_pitch_link: mass 0.087149 -> 0.084987
- link L_foot_link: mass 1.0326 -> 1.0304
- link L_hip_pitch_link: mass 2.1718 -> 2.1738
- link L_hip_roll_link: mass 1.6093 -> 1.6181
- link L_thigh_link: mass 2.8959 -> 2.9294
- link R_ankle_pitch_link: mass 0.087149 -> 0.084987
- link R_foot_link: mass 1.0326 -> 1.0304
- link R_hip_pitch_link: mass 2.1718 -> 2.1738
- link R_hip_roll_link: mass 1.6093 -> 1.6181
- link R_thigh_link: mass 2.8959 -> 2.9294
- link base_link: mass 27.461 -> 5.1659
Joints:
- added joint L_shoulder_pitch_joint: type revolute, parent torso_link, child L_shoulder_pitch_link, origin xyz=-0.015 -0.2 0.3625 rpy=0 0 0, axis 0 1 0, limit lower=-3.141592653589793 upper=1.0471975511965976 effort=60 velocity=20
- added joint L_shoulder_roll_joint: type revolute, parent L_shoulder_pitch_link, child L_arm_link, origin xyz=0 0 0 rpy=0 0 0, axis 1 0 0, limit lower=-0.5585053606381855 upper=0.5235987755982988 effort=60 velocity=20
- added joint R_shoulder_pitch_joint: type revolute, parent torso_link, child R_shoulder_pitch_link, origin xyz=-0.015 0.2 0.3625 rpy=0 0 0, axis 0 1 0, limit lower=-3.141592653589793 upper=1.0471975511965976 effort=60 velocity=20
- added joint R_shoulder_roll_joint: type revolute, parent R_shoulder_pitch_link, child R_arm_link, origin xyz=0 0 0 rpy=0 0 0, axis -1 0 0, limit lower=-0.5585053606381855 upper=0.5235987755982988 effort=60 velocity=20
- added joint waist_yaw_joint: type revolute, parent base_link, child torso_link, origin xyz=0 0 0.1175 rpy=0 0 0, axis 0 0 1, limit lower=-1.0471975511965976 upper=1.0471975511965976 effort=120 velocity=20
- joint L_ankle_pitch_joint: limit lower=-0.872665 upper=0.523599 effort=90 velocity=20 -> lower=-0.8726646259971648 upper=0.5235987755982988 effort=90 velocity=20
- joint L_ankle_roll_joint: limit lower=-0.349066 upper=0.349066 effort=50 velocity=20 -> lower=-0.3490658503988659 upper=0.3490658503988659 effort=50 velocity=20
- joint L_hip_pitch_joint: limit lower=-2.18166 upper=0.523599 effort=120 velocity=20 -> lower=-2.0943951023931953 upper=0.4537856055185257 effort=120 velocity=20
- joint L_hip_roll_joint: limit lower=-0.785398 upper=0.436332 effort=120 velocity=20 -> lower=-0.7853981633974483 upper=0.4363323129985824 effort=120 velocity=20
- joint L_hip_yaw_joint: limit lower=-0.872665 upper=0.872665 effort=60 velocity=20 -> lower=-0.8203047484373349 upper=0.8901179185171081 effort=60 velocity=20
- joint L_knee_joint: limit lower=-2.094395 upper=0.0 effort=120 velocity=20 -> lower=-2.0943951023931953 upper=0.0 effort=120 velocity=20
- joint R_ankle_pitch_joint: limit lower=-0.872665 upper=0.523599 effort=90 velocity=20 -> lower=-0.8726646259971648 upper=0.5235987755982988 effort=90 velocity=20
- joint R_ankle_roll_joint: limit lower=-0.349066 upper=0.349066 effort=50 velocity=20 -> lower=-0.3490658503988659 upper=0.3490658503988659 effort=50 velocity=20
- joint R_hip_pitch_joint: limit lower=-2.18166 upper=0.523599 effort=120 velocity=20 -> lower=-2.0943951023931953 upper=0.4537856055185257 effort=120 velocity=20
- joint R_hip_roll_joint: limit lower=-0.785398 upper=0.436332 effort=120 velocity=20 -> lower=-0.7853981633974483 upper=0.4363323129985824 effort=120 velocity=20
- joint R_hip_yaw_joint: limit lower=-0.872665 upper=0.872665 effort=60 velocity=20 -> lower=-0.8203047484373349 upper=0.8901179185171081 effort=60 velocity=20
- joint R_knee_joint: limit lower=-2.094395 upper=0.0 effort=120 velocity=20 -> lower=-2.0943951023931953 upper=0.0 effort=120 velocity=20

Commit message: a switched-off light bulb is not suppression: 69 pelvis screws were missing from the viewer AND from the mass model
Reported as "the CenterParts screws are gone from the viewer". They were gone from the mass
model too, and for the same reason: Fusion's `live` flag was read as "not part of the robot",
and two very different things wear that flag.

  alternatives   ArmR_fullDoF, Actuators-NotUse, Human_Solid (REF)   25 bodies, 671.044 kg
  merely hidden  every fastener inside CenterParts                   69 bodies,   0.201 kg

The first must be excluded; the second is real hardware switched off so the parts underneath
can be seen. The split is made on branch name and was verified against the dump rather than
assumed: the test matches 25 hidden bodies and ZERO live ones, and every hidden body it does
not match is a fastener on a fully visible sub-assembly. The screws are modelled on both sides
(41 left / 2 centre / 26 right in CAD x), so they count as-is with no mirroring.

  pelvis 5.166 -> 5.367 kg, whole robot 42.098 -> 42.299 kg, revalidated

Also: 66 fasteners whose path carries no group - 21 loose root-level occurrences and the 45
under Ankle2Feet - had no link at all and displayed as "?". They are now assigned to the
nearest link mesh, at match distances around 2 mm, so nothing is ambiguous.

The viewer flags CAD-hidden fasteners and can filter them: someone looking at the pelvis
should be told those 69 screws are switched off in the CAD they have open, not shown them
silently as if nothing were different.

Two "missing from the viewer" reports in a row have now each exposed a real defect. The
visualisation is not decoration, it is the check.

Co-Authored-By: Claude Opus 4.8 <noreply@anthropic.com>

File: pygmalion_locomotion/assets/pygmalion_v2/pygmalion_v2.urdf (robot description, URDF)
Before this commit: robot pygmalion_v2, 18 links, 17 joints
Links:
- link base_link: mass 5.1659 -> 5.3668

Commit message: hip limits: the -45 abduction cap had no basis, and the sweep never found the real stop
The ROM table called hip_roll abduction -45 a "design cap". It was not. -45 is the old
pygmalion.xml range carried over untouched, and nothing in docs records a decision about
abduction - only the +25 adduction verdict. The brief was "hip pitch roll yaw knee are all
wrong, set them from where the parts actually collide", so keeping the exact number that was
called wrong and relabelling it as a design decision was the worst of both.

The measurement was complicit: hip_roll was swept only to -70, hit nothing, and reported
"-70" - a search boundary read as a limit. Widened to -120 the abduction stop is -86, both
sides now blocked by hip_pitch_link ~ hip_roll_link.

Limits set by the user, each inside the measured stop (the build asserts this):

  hip_pitch  -120 / +25    metal at +26
  hip_roll    -85 / +25    metal at -86, adduction from the gen21 verdict
  hip_yaw     -45 / +45    metal at -48 / +52

Two robustness fixes so this class of error is harder to repeat: rom_check.py MERGES into
rom_measured.json instead of overwriting it - re-measuring one joint had just wiped the other
eight, after which build_robot silently used inherited ranges - and a joint that hits nothing
inside its span is reported as a search boundary, not a limit.

Revalidated: 42.299 kg, L/R conventions unchanged, seven of nine joints with zero self-contact
over their full range; the two that remain are the dummy arm against the thigh (docs/88 s3c).

Co-Authored-By: Claude Opus 4.8 <noreply@anthropic.com>

File: pygmalion_locomotion/assets/pygmalion_v2/pygmalion_v2.urdf (robot description, URDF)
Before this commit: robot pygmalion_v2, 18 links, 17 joints
Joints:
- joint L_hip_pitch_joint: limit lower=-2.0943951023931953 upper=0.4537856055185257 effort=120 velocity=20 -> lower=-2.0943951023931953 upper=0.4363323129985824 effort=120 velocity=20
- joint L_hip_roll_joint: limit lower=-0.7853981633974483 upper=0.4363323129985824 effort=120 velocity=20 -> lower=-1.4835298641951802 upper=0.4363323129985824 effort=120 velocity=20
- joint L_hip_yaw_joint: limit lower=-0.8203047484373349 upper=0.8901179185171081 effort=60 velocity=20 -> lower=-0.7853981633974483 upper=0.7853981633974483 effort=60 velocity=20
- joint R_hip_pitch_joint: limit lower=-2.0943951023931953 upper=0.4537856055185257 effort=120 velocity=20 -> lower=-2.0943951023931953 upper=0.4363323129985824 effort=120 velocity=20
- joint R_hip_roll_joint: limit lower=-0.7853981633974483 upper=0.4363323129985824 effort=120 velocity=20 -> lower=-1.4835298641951802 upper=0.4363323129985824 effort=120 velocity=20
- joint R_hip_yaw_joint: limit lower=-0.8203047484373349 upper=0.8901179185171081 effort=60 velocity=20 -> lower=-0.7853981633974483 upper=0.7853981633974483 effort=60 velocity=20
