Commit message: loop ankle: red team (3 confirmed of 7), loop URDF carries the crank/rod tree, ground video with the leg held
- docs/91: nv is 35 in the XML and 30 in the training spec (upper body welded), not '30'
  everywhere; PYG_UPPER_DOF=1 crosses mjwarp's nv>32 sparse threshold. Transmission
  numbers were from the soft-constraint run (-1.167/-1.348); the stiff rod ends give
  -1.21/-1.42, matching the mjlab hanging test. Red-team section added.
- build_robot: the loop URDF now contains crank -> 1 g dummy -> rod as revolute chains
  (URDF has neither universal joints nor loop closure; the closure is a comment). Before
  this the loop URDF was the serial tree with the loop model's lighter shin - 0.43 kg of
  cranks and rods simply missing.
- urdf_crosscheck: unlimited MJCF hinges are not range-compared (URDF must write +-pi);
  URDF-only bodies are reported. Loop model: MATCH, 29/29 joints, 0.0000 mm over 200
  random poses, 4 dummy links reported.
- loop_ankle_verify ground test: hips/knees held by PD (they hung off the pinned base
  before), sole 2 mm above the floor so a crank tilt brings the toe/heel edge into
  contact: 0-3 contacts, 0-128 N, closure 0.002 mm.

Co-Authored-By: Claude Opus 5 <noreply@anthropic.com>

File: pygmalion_locomotion/assets/pygmalion_v2/pygmalion_v3_printed_loop.urdf (robot description, URDF)
Before this commit: robot pygmalion_v3_printed_loop, 18 links, 17 joints
Links:
- added link L_crank_A, mass 0.034678; visual mesh filename=meshes/crank_A.stl
- added link L_crank_B, mass 0.033884; visual mesh filename=meshes/crank_B.stl
- added link L_rod_A, mass 0.080611; visual mesh filename=meshes/rod_A.stl
- added link L_rod_A_u, mass 0.001
- added link L_rod_B, mass 0.064627; visual mesh filename=meshes/rod_B.stl
- added link L_rod_B_u, mass 0.001
- added link R_crank_A, mass 0.034678; visual mesh filename=meshes/R_crank_A.stl
- added link R_crank_B, mass 0.033884; visual mesh filename=meshes/R_crank_B.stl
- added link R_rod_A, mass 0.080611; visual mesh filename=meshes/R_rod_A.stl
- added link R_rod_A_u, mass 0.001
- added link R_rod_B, mass 0.064627; visual mesh filename=meshes/R_rod_B.stl
- added link R_rod_B_u, mass 0.001
Joints:
- added joint L_crank_A_joint: type revolute, parent L_shin_link, child L_crank_A, origin xyz=-0.029945 -0.001718 -0.190034 rpy=0 0 0, axis 0.0000 1.0000 0.0000, limit lower=-1.2 upper=1.2 effort=60.0 velocity=20
- added joint L_crank_B_joint: type revolute, parent L_shin_link, child L_crank_B, origin xyz=-0.030055 0.001717 -0.290034 rpy=0 0 0, axis 0.0000 1.0000 0.0000, limit lower=-1.2 upper=1.2 effort=60.0 velocity=20
- added joint L_rod_A_u1: type revolute, parent L_crank_A, child L_rod_A_u, origin xyz=-0.061494 0.042718 -0.021185 rpy=0 0 0, axis 0.0000 1.0000 0.0000, limit lower=-3.1416 upper=3.1416 effort=0 velocity=50
- added joint L_rod_A_u2: type revolute, parent L_rod_A_u, child L_rod_A, origin xyz=0 0 0 rpy=0 0 0, axis -0.9993 0.0000 -0.0379, limit lower=-3.1416 upper=3.1416 effort=0 velocity=50
- added joint L_rod_B_u1: type revolute, parent L_crank_B, child L_rod_B_u, origin xyz=-0.060039 -0.042717 -0.01522 rpy=0 0 0, axis 0.0000 1.0000 0.0000, limit lower=-3.1416 upper=3.1416 effort=0 velocity=50
- added joint L_rod_B_u2: type revolute, parent L_rod_B_u, child L_rod_B, origin xyz=0 0 0 rpy=0 0 0, axis -0.9988 0.0000 -0.0492, limit lower=-3.1416 upper=3.1416 effort=0 velocity=50
- added joint R_crank_A_joint: type revolute, parent R_shin_link, child R_crank_A, origin xyz=-0.029945 0.001718 -0.190034 rpy=0 0 0, axis 0.0000 1.0000 0.0000, limit lower=-1.2 upper=1.2 effort=60.0 velocity=20
- added joint R_crank_B_joint: type revolute, parent R_shin_link, child R_crank_B, origin xyz=-0.030055 -0.001717 -0.290034 rpy=0 0 0, axis 0.0000 1.0000 0.0000, limit lower=-1.2 upper=1.2 effort=60.0 velocity=20
- added joint R_rod_A_u1: type revolute, parent R_crank_A, child R_rod_A_u, origin xyz=-0.061494 -0.042718 -0.021185 rpy=0 0 0, axis 0.0000 1.0000 0.0000, limit lower=-3.1416 upper=3.1416 effort=0 velocity=50
- added joint R_rod_A_u2: type revolute, parent R_rod_A_u, child R_rod_A, origin xyz=0 0 0 rpy=0 0 0, axis -0.9993 0.0000 -0.0379, limit lower=-3.1416 upper=3.1416 effort=0 velocity=50
- added joint R_rod_B_u1: type revolute, parent R_crank_B, child R_rod_B_u, origin xyz=-0.060039 0.042717 -0.01522 rpy=0 0 0, axis 0.0000 1.0000 0.0000, limit lower=-3.1416 upper=3.1416 effort=0 velocity=50
- added joint R_rod_B_u2: type revolute, parent R_rod_B_u, child R_rod_B, origin xyz=0 0 0 rpy=0 0 0, axis -0.9988 0.0000 -0.0492, limit lower=-3.1416 upper=3.1416 effort=0 velocity=50
